Commit message: updated urdf

File: spot_arm_description/urdf/spot_arm.xacro (robot description, xacro)
@@ -4,5 +4,5 @@
 <xacro:include filename="$(find spot_arm_description)/urdf/spot_arm.trans" />
 <xacro:include filename="$(find spot_arm_description)/urdf/spot_arm.gazebo" />
-<link name="base_link">
+<link name="base">
   <inertial>
     <origin rpy="0 0 0" xyz="1.2371844231029972e-17 0.0 0.0325"/>
@@ -194,5 +194,5 @@
 <joint name="Rev9" type="revolute">
   <origin rpy="0 0 0" xyz="0.0 0.0 0.065"/>
-  <parent link="base_link"/>
+  <parent link="base"/>
   <child link="Part0_1"/>
   <axis xyz="0.0 0.0 1.0"/>
